File: snowpixel.kicad_pcb (KiCad board)
At the start: 2 copper layers, 19.9 x 19.9 mm, 112 parts, among them J1 Conn_01x01_Pin, J10 Conn_01x01_Pin, J11 Conn_01x01_Pin, J13 Conn_01x01_Pin, J15 Conn_01x01_Pin, J17 Conn_01x01_Pin, J18 Conn_01x01_Pin, J2 Conn_01x01_Pin, J21 Conn_01x01_Pin, J22 Conn_01x01_Pin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

Commit message: Change silkscreen text
Other:
- board text added: "Nora"
- board text added: "SnowPixel"
- board text removed: "nora"
- board text removed: "snowpixel"
Changed lines of the file:
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@@
 		)
 	)
-	(gr_text "nora"
+	(gr_text "Nora"
 		(at 126.16 59.81 90)
 		(layer "B.SilkS")
@@
 		)
 	)
-	(gr_text "snowpixel"
-		(at 111.7 60.45 90)
+	(gr_text "SnowPixel"
+		(at 111.8 60.5 90)
 		(layer "B.SilkS")
 		(effects
